Commit message: modified mrp package to use arduino_interface

File: src/jetson/dev_ws/src/mrp/description/robot.urdf.xacro (robot description, xacro)
@@ -1,4 +1,5 @@
 <?xml version="1.0"?>
 <robot xmlns:xacro="http://www.ros.org/wiki/xacro"  name="robot">
+    <xacro:arg name="sim_mode" default="false"/>
     <!-- TODO: update measurements -->
     <!-- These are in meters and kilograms -->

File: src/jetson/dev_ws/src/mrp/description/ros2_control.xacro (robot description, xacro)
@@ -1,44 +1,95 @@
 <?xml version="1.0"?>
 <robot xmlns:xacro="http://www.ros.org/wiki/xacro">
-    <ros2_control name="GazeboSystem" type="system">
-        <hardware>
-            <plugin>gazebo_ros2_control/GazeboSystem</plugin>
-        </hardware>
-        <joint name="rear_left_wheel_joint">
-            <command_interface name="velocity">
-                <param name="min">-10</param>
-                <param name="max">10</param>
-            </command_interface>
-            <state_interface name="velocity"/>
-            <state_interface name="position"/>
-        </joint>
-        <joint name="rear_right_wheel_joint">
-            <command_interface name="velocity">
-                <param name="min">-10</param>
-                <param name="max">10</param>
-            </command_interface>
-            <state_interface name="velocity"/>
-            <state_interface name="position"/>
-        </joint>
-        <joint name="front_left_wheel_joint">
-            <command_interface name="velocity">
-                <param name="min">-10</param>
-                <param name="max">10</param>
-            </command_interface>
-            <state_interface name="velocity"/>
-            <state_interface name="position"/>
-        </joint>
-        <joint name="front_right_wheel_joint">
-            <command_interface name="velocity">
-                <param name="min">-10</param>
-                <param name="max">10</param>
-            </command_interface>
-            <state_interface name="velocity"/>
-            <state_interface name="position"/>
-        </joint>
-    </ros2_control>
+    <xacro:unless value="$(arg sim_mode)">
+        <ros2_control name="RealRobot" type="system">
+            <hardware>
+                <plugin>arduino_interface/ArduinoInterface</plugin>
+                <param name="rl_wheel_name">rear_left_wheel_joint</param>
+                <param name="rr_wheel_name">rear_right_wheel_joint</param>
+                <param name="fl_wheel_name">front_left_wheel_joint</param>
+                <param name="fr_wheel_name">front_right_wheel_joint</param>
+                <param name="loop_rate">30</param>
+                <param name="device">/dev/ttyUSB0</param> <!-- TODO -->
+                <param name="baud_rate">57600</param>
+                <param name="timeout">1000</param>
+                <param name="enc_counts_per_rev">30</param>
+            </hardware>
+            <joint name="rear_left_wheel_joint">
+                <command_interface name="velocity">
+                    <param name="min">-10</param>
+                    <param name="max">10</param>
+                </command_interface>
+                <state_interface name="velocity"/>
+                <state_interface name="position"/>
+            </joint>
+            <joint name="rear_right_wheel_joint">
+                <command_interface name="velocity">
+                    <param name="min">-10</param>
+                    <param name="max">10</param>
+                </command_interface>
+                <state_interface name="velocity"/>
+                <state_interface name="position"/>
+            </joint>
+            <joint name="front_left_wheel_joint">
+                <command_interface name="velocity">
+                    <param name="min">-10</param>
+                    <param name="max">10</param>
+                </command_interface>
+                <state_interface name="velocity"/>
+                <state_interface name="position"/>
+            </joint>
+            <joint name="front_right_wheel_joint">
+                <command_interface name="velocity">
+                    <param name="min">-10</param>
+                    <param name="max">10</param>
+                </command_interface>
+                <state_interface name="velocity"/>
+                <state_interface name="position"/>
+            </joint>
+        </ros2_control>
+    </xacro:unless>
+    <xacro:if value="$(arg sim_mode)">
+        <ros2_control name="GazeboSystem" type="system">
+            <hardware>
+                <plugin>gazebo_ros2_control/GazeboSystem</plugin>
+            </hardware>
+            <joint name="rear_left_wheel_joint">
+                <command_interface name="velocity">
+                    <param name="min">-10</param>
+                    <param name="max">10</param>
+                </command_interface>
+                <state_interface name="velocity"/>
+                <state_interface name="position"/>
+            </joint>
+            <joint name="rear_right_wheel_joint">
+                <command_interface name="velocity">
+                    <param name="min">-10</param>
+                    <param name="max">10</param>
+                </command_interface>
+                <state_interface name="velocity"/>
+                <state_interface name="position"/>
+            </joint>
+            <joint name="front_left_wheel_joint">
+                <command_interface name="velocity">
+                    <param name="min">-10</param>
+                    <param name="max">10</param>
+                </command_interface>
+                <state_interface name="velocity"/>
+                <state_interface name="position"/>
+            </joint>
+            <joint name="front_right_wheel_joint">
+                <command_interface name="velocity">
+                    <param name="min">-10</param>
+                    <param name="max">10</param>
+                </command_interface>
+                <state_interface name="velocity"/>
+                <state_interface name="position"/>
+            </joint>
+        </ros2_control>
+    </xacro:if>
     <gazebo>
         <plugin name="gazebo_ros2_control" filename="libgazebo_ros2_control.so">
             <parameters>$(find mrp)/config/my_controllers.yaml</parameters>
+            <parameters>$(find mrp)/config/gaz_ros2_ctl_use_sim.yaml</parameters>
         </plugin>
     </gazebo>

Commit message: updated robot dimensions

File: src/jetson/dev_ws/src/mrp/description/robot.urdf.xacro (robot description, xacro)
@@ -2,22 +2,23 @@
 <robot xmlns:xacro="http://www.ros.org/wiki/xacro"  name="robot">
     <xacro:arg name="sim_mode" default="false"/>
-    <!-- TODO: update measurements -->
     <!-- These are in meters and kilograms -->
     <xacro:property name="chassis_length" value="0.4"/>
     <xacro:property name="chassis_width" value="0.35"/>
-    <xacro:property name="chassis_height" value="0.25"/>
-    <xacro:property name="chassis_mass" value="30"/>
+    <xacro:property name="chassis_height" value="0.28"/>
+    <xacro:property name="chassis_mass" value="30"/> <!-- TODO -->
     <xacro:property name="wheel_radius" value="0.0762"/>
-    <xacro:property name="wheel_thickness" value="0.05"/>
-    <xacro:property name="wheel_mass" value="0.5"/>
-    <xacro:property name="wheel_offset_x" value="0.1"/>
-    <xacro:property name="wheel_offset_y" value="0.175"/>
-    <xacro:property name="wheel_offset_z" value="0"/>
+    <xacro:property name="wheel_thickness" value="0.0381"/>
+    <xacro:property name="wheel_mass" value="1.5"/> <!-- TODO -->
+    <!-- From bottom center -->
+    <xacro:property name="wheel_offset_x" value="0.0875"/>
+    <xacro:property name="wheel_offset_y" value="0.1877"/>
+    <xacro:property name="wheel_offset_z" value="0.0508"/>
     <xacro:property name="lidar_radius" value="0.035"/>
     <xacro:property name="lidar_thickness" value="0.02"/>
     <xacro:property name="lidar_mass" value="0.5"/>
-    <xacro:property name="lidar_offset_x" value="0.3"/>
+    <!-- From bottom rear --> <!-- TODO -->
+    <xacro:property name="lidar_offset_x" value="0.3246"/>
     <xacro:property name="lidar_offset_y" value="0"/>
-    <xacro:property name="lidar_offset_z" value="0.25"/>
+    <xacro:property name="lidar_offset_z" value="0.31175"/>
     <xacro:include filename="mrp_core.xacro"/>
     <xacro:include filename="ros2_control.xacro"/>

Commit message: corrected wheel positioning

File: src/jetson/dev_ws/src/mrp/description/robot.urdf.xacro (robot description, xacro)
@@ -12,5 +12,5 @@
     <!-- From bottom center -->
     <xacro:property name="wheel_offset_x" value="0.0875"/>
-    <xacro:property name="wheel_offset_y" value="0.1877"/>
+    <xacro:property name="wheel_offset_y" value="${0.1877 + wheel_thickness/2}"/>
     <xacro:property name="wheel_offset_z" value="0.0508"/>
     <xacro:property name="lidar_radius" value="0.035"/>
