Commit message: corrected bug with launch Command substitution

File: src/jetson/dev_ws/src/mrp/description/lidar.xacro (robot description, xacro)
@@ -1,4 +1,12 @@
 <?xml version="1.0"?>
 <robot xmlns:xacro="http://www.ros.org/wiki/xacro">
+    <!-- These are in meters and kilograms -->
+    <xacro:property name="lidar_radius" value="0.035"/>
+    <xacro:property name="lidar_thickness" value="0.02"/>
+    <xacro:property name="lidar_mass" value="0.5"/>
+    <!-- From bottom rear --> <!-- TODO -->
+    <xacro:property name="lidar_offset_x" value="0.3246"/>
+    <xacro:property name="lidar_offset_y" value="0"/>
+    <xacro:property name="lidar_offset_z" value="0.31175"/>
     <joint name="laser_joint" type="fixed">
         <parent link="chassis"/>

File: src/jetson/dev_ws/src/mrp/description/mrp_core.xacro (robot description, xacro)
@@ -2,4 +2,16 @@
 <robot xmlns:xacro="http://www.ros.org/wiki/xacro">
     <xacro:include filename="inertial_macros.xacro"/>
+    <!-- These are in meters and kilograms -->
+    <xacro:property name="chassis_length" value="0.4"/>
+    <xacro:property name="chassis_width" value="0.35"/>
+    <xacro:property name="chassis_height" value="0.28"/>
+    <xacro:property name="chassis_mass" value="30"/> <!-- TODO -->
+    <xacro:property name="wheel_radius" value="0.0762"/>
+    <xacro:property name="wheel_thickness" value="0.0381"/>
+    <xacro:property name="wheel_mass" value="1.5"/> <!-- TODO -->
+    <!-- From bottom center -->
+    <xacro:property name="wheel_offset_x" value="0.0875"/>
+    <xacro:property name="wheel_offset_y" value="${0.1877 + wheel_thickness/2}"/>
+    <xacro:property name="wheel_offset_z" value="0.0508"/>
     <!-- Material setup for simulation -->
     <material name="white">
@@ -22,5 +34,5 @@
         <parent link="base_link"/>
         <child link="chassis"/>
-        <origin xyz="-${chassis_length/2} 0 0"/> <!-- TODO: difference to from center of turning to rear of robot -->
+        <origin xyz="-${chassis_length/2} 0 0"/>
     </joint>
     <link name="chassis">

File: src/jetson/dev_ws/src/mrp/description/robot.urdf.xacro (robot description, xacro)
@@ -1,26 +1,13 @@
 <?xml version="1.0"?>
 <robot xmlns:xacro="http://www.ros.org/wiki/xacro"  name="robot">
+    <xacro:arg name="use_ros2_control" default="true"/>
     <xacro:arg name="sim_mode" default="false"/>
-    <!-- These are in meters and kilograms -->
-    <xacro:property name="chassis_length" value="0.4"/>
-    <xacro:property name="chassis_width" value="0.35"/>
-    <xacro:property name="chassis_height" value="0.28"/>
-    <xacro:property name="chassis_mass" value="30"/> <!-- TODO -->
-    <xacro:property name="wheel_radius" value="0.0762"/>
-    <xacro:property name="wheel_thickness" value="0.0381"/>
-    <xacro:property name="wheel_mass" value="1.5"/> <!-- TODO -->
-    <!-- From bottom center -->
-    <xacro:property name="wheel_offset_x" value="0.0875"/>
-    <xacro:property name="wheel_offset_y" value="${0.1877 + wheel_thickness/2}"/>
-    <xacro:property name="wheel_offset_z" value="0.0508"/>
-    <xacro:property name="lidar_radius" value="0.035"/>
-    <xacro:property name="lidar_thickness" value="0.02"/>
-    <xacro:property name="lidar_mass" value="0.5"/>
-    <!-- From bottom rear --> <!-- TODO -->
-    <xacro:property name="lidar_offset_x" value="0.3246"/>
-    <xacro:property name="lidar_offset_y" value="0"/>
-    <xacro:property name="lidar_offset_z" value="0.31175"/>
     <xacro:include filename="mrp_core.xacro"/>
-    <xacro:include filename="ros2_control.xacro"/>
+    <xacro:if value="$(arg use_ros2_control)">
+        <xacro:include filename="ros2_control.xacro" />
+    </xacro:if>
+    <xacro:unless value="$(arg use_ros2_control)">
+        <xacro:include filename="gazebo_control.xacro" />
+    </xacro:unless>
     <xacro:include filename="lidar.xacro"/>
 </robot>

Commit message: corrected lidar position

File: src/jetson/dev_ws/src/mrp/description/lidar.xacro (robot description, xacro)
@@ -8,5 +8,5 @@
     <xacro:property name="lidar_offset_x" value="0.3246"/>
     <xacro:property name="lidar_offset_y" value="0"/>
-    <xacro:property name="lidar_offset_z" value="0.31175"/>
+    <xacro:property name="lidar_offset_z" value="${0.31175 + lidar_thickness/2}"/>
     <joint name="laser_joint" type="fixed">
         <parent link="chassis"/>
