Commit message: corrected wheel offsets

File: src/jetson/dev_ws/src/mrp/description/mrp_core.xacro (robot description, xacro)
@@ -61,5 +61,5 @@
         <parent link="base_link"/>
         <child link="rear_left_wheel"/>
-        <origin xyz="${-wheel_offset_x} ${-wheel_offset_y} ${wheel_offset_z}" rpy="-${pi/2} 0 0"/> <!-- Rotate to be upright -->
+        <origin xyz="${-wheel_offset_x} ${wheel_offset_y} ${wheel_offset_z}" rpy="-${pi/2} 0 0"/> <!-- Rotate to be upright -->
         <axis xyz="0 0 1"/> <!-- Direction of rotation -->
     </joint>
@@ -87,5 +87,5 @@
         <parent link="base_link"/>
         <child link="rear_right_wheel"/>
-        <origin xyz="${-wheel_offset_x} ${wheel_offset_y} ${wheel_offset_z}" rpy="${pi/2} 0 0"/>
+        <origin xyz="${-wheel_offset_x} ${-wheel_offset_y} ${wheel_offset_z}" rpy="${pi/2} 0 0"/>
         <axis xyz="0 0 -1"/>
     </joint>
@@ -113,5 +113,5 @@
         <parent link="base_link"/>
         <child link="front_left_wheel"/>
-        <origin xyz="${wheel_offset_x} ${-wheel_offset_y} ${wheel_offset_z}" rpy="-${pi/2} 0 0"/>
+        <origin xyz="${wheel_offset_x} ${wheel_offset_y} ${wheel_offset_z}" rpy="-${pi/2} 0 0"/>
         <axis xyz="0 0 1"/>
     </joint>
@@ -139,5 +139,5 @@
         <parent link="base_link"/>
         <child link="front_right_wheel"/>
-        <origin xyz="${wheel_offset_x} ${wheel_offset_y} ${wheel_offset_z}" rpy="${pi/2} 0 0"/>
+        <origin xyz="${wheel_offset_x} ${-wheel_offset_y} ${wheel_offset_z}" rpy="${pi/2} 0 0"/>
         <axis xyz="0 0 -1"/>
     </joint>

Commit message: added SLAM

File: src/jetson/dev_ws/src/mrp/description/mrp_core.xacro (robot description, xacro)
@@ -29,4 +29,12 @@
     <!-- Base link -->
     <link name="base_link">
+    </link>
+    <!-- Base footprint link -->
+    <joint name="base_footprint_joint" type="fixed">
+        <parent link="base_link"/>
+        <child link="base_footprint"/>
+        <origin xyz="0 0 0"/>
+    </joint>
+    <link name="base_footprint">
     </link>
     <!-- Chassis -->
